File: src/AirQualitySensor/PCB_Files_KiCad/AirQualitySensorBreakOutBoard/AirQualitySensorBreakOutBoard.kicad_pcb (KiCad board)
At the start: 2 copper layers, 113.8 x 36 mm, 24 parts, among them J1 Conn_01x02_Male, J2 Conn_01x02_Male, J3 Conn_01x02_Male, J4 Conn_01x07_Male, Q1 IRLB8721PBF, U1 PMS5003, U2 PMS5003, U3 SPS30, U4 SHT31, U6 lilygo-ttgo-t-sim7000g-esp32-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

Commit message: update
Routing:
- net 5V0: track 106.0 -> 107.2 mm
- net VDD2: track 159.7 -> 160.8 mm
Changed lines of the file:
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@@
       (drillshape 0)
       (scaleselection 1)
-      (outputdirectory "C:/Users/seand/OneDrive/Desktop/AirQualitySensorPCB_FlatCam/")
+      (outputdirectory "C:/Users/seand/OneDrive/Desktop/AQS Gerber files/")
     )
   )
@@
   (segment (start 55.1 26.5) (end 52.5 29.1) (width 1) (layer "F.Cu") (net 1))
   (segment (start 51.99 30.71) (end 51.99 33.7) (width 1) (layer "F.Cu") (net 1))
+  (segment (start 67.6 27.882379) (end 66.017621 27.882379) (width 1) (layer "F.Cu") (net 2))
+  (segment (start 80.7 37.3) (end 83.5 34.5) (width 1) (layer "F.Cu") (net 2))
   (segment (start 29.4 26.435001) (end 29.53 26.565001) (width 1) (layer "F.Cu") (net 2))
+  (segment (start 63.7 17.7) (end 62.8 18.6) (width 1) (layer "F.Cu") (net 2))
   (segment (start 19.7 41.9) (end 21.4 43.6) (width 1) (layer "F.Cu") (net 2))
-  (segment (start 70.3 33.5) (end 74.1 37.3) (width 1) (layer "F.Cu") (net 2))
-  (segment (start 79.96 37.3) (end 82.66 34.6) (width 1) (layer "F.Cu") (net 2))
-  (segment (start 82.66 34.6) (end 82.66 19.36) (width 1) (layer "F.Cu") (net 2))
+  (segment (start 65.1 31) (end 67.6 33.5) (width 1) (layer "F.Cu") (net 2))
   (segment (start 19.7 37.8) (end 19.7 41.9) (width 1) (layer "F.Cu") (net 2))
   (segment (start 30.03 32.865) (end 30.03 34.07) (width 1) (layer "F.Cu") (net 2))
   (segment (start 55.04 34.96) (end 52.35 37.65) (width 1) (layer "F.Cu") (net 2))
-  (segment (start 63.7 17.7) (end 62.8 18.6) (width 1) (layer "F.Cu") (net 2))
+  (segment (start 67.6 33.5) (end 70.3 33.5) (width 1) (layer "F.Cu") (net 2))
   (segment (start 50.02 21.78) (end 48.7 23.1) (width 1) (layer "F.Cu") (net 2))
   (segment (start 29.4 26.435001) (end 26.861488 26.435001) (width 1) (layer "F.Cu") (net 2))
@@
   (segment (start 24.25 41.35) (end 24.25 40.865) (width 1) (layer "F.Cu") (net 2))
   (segment (start 20.7 36.8) (end 19.7 37.8) (width 1) (layer "F.Cu") (net 2))
-  (segment (start 67.6 33.5) (end 70.3 33.5) (width 1) (layer "F.Cu") (net 2))
   (segment (start 52.35 40.88) (end 52.415126 40.88) (width 1) (layer "F.Cu") (net 2))
+  (segment (start 81 17.7) (end 63.7 17.7) (width 1) (layer "F.Cu") (net 2))
   (segment (start 21.4 43.6) (end 22 43.6) (width 1) (layer "F.Cu") (net 2))
-  (segment (start 66.017621 27.882379) (end 65.1 28.8) (width 1) (layer "F.Cu") (net 2))
+  (segment (start 65.1 28.8) (end 65.1 31) (width 1) (layer "F.Cu") (net 2))
   (segment (start 67.6 27.882379) (end 57.357621 27.882379) (width 1) (layer "F.Cu") (net 2))
-  (segment (start 67.6 27.882379) (end 66.017621 27.882379) (width 1) (layer "F.Cu") (net 2))
   (segment (start 62.7 18.6) (end 51.492234 18.6) (width 1) (layer "F.Cu") (net 2))
   (segment (start 51.492234 18.6) (end 50.02 20.072234) (width 1) (layer "F.Cu") (net 2))
-  (segment (start 65.1 28.8) (end 65.1 31) (width 1) (layer "F.Cu") (net 2))
   (segment (start 50.02 20.072234) (end 50.02 20.5) (width 1) (layer "F.Cu") (net 2))
   (segment (start 55.04 30.2) (end 55.04 34.96) (width 1) (layer "F.Cu") (net 2))
+  (segment (start 74.1 37.3) (end 80.7 37.3) (width 1) (layer "F.Cu") (net 2))
   (segment (start 29.53 26.565001) (end 29.53 32.365) (width 1) (layer "F.Cu") (net 2))
   (segment (start 52.35 37.65) (end 52.35 40.88) (width 1) (layer "F.Cu") (net 2))
+  (segment (start 83.5 20.2) (end 81 17.7) (width 1) (layer "F.Cu") (net 2))
   (segment (start 29.5 24.4) (end 29.4 24.5) (width 1) (layer "F.Cu") (net 2))
   (segment (start 33.9 24.4) (end 29.5 24.4) (width 1) (layer "F.Cu") (net 2))
-  (segment (start 82.66 19.36) (end 81 17.7) (width 1) (layer "F.Cu") (net 2))
-  (segment (start 81 17.7) (end 63.7 17.7) (width 1) (layer "F.Cu") (net 2))
+  (segment (start 83.5 34.5) (end 83.5 20.2) (width 1) (layer "F.Cu") (net 2))
+  (segment (start 70.3 33.5) (end 74.1 37.3) (width 1) (layer "F.Cu") (net 2))
+  (segment (start 66.017621 27.882379) (end 65.1 28.8) (width 1) (layer "F.Cu") (net 2))
   (segment (start 35.2 23.1) (end 33.9 24.4) (width 1) (layer "F.Cu") (net 2))
   (segment (start 22 43.6) (end 24.25 41.35) (width 1) (layer "F.Cu") (net 2))
-  (segment (start 65.1 31) (end 67.6 33.5) (width 1) (layer "F.Cu") (net 2))
   (segment (start 30.03 34.07) (end 27.3 36.8) (width 1) (layer "F.Cu") (net 2))
-  (segment (start 74.1 37.3) (end 79.96 37.3) (width 1) (layer "F.Cu") (net 2))
   (segment (start 29.53 32.365) (end 30.03 32.865) (width 1) (layer "F.Cu") (net 2))
   (segment (start 57.357621 27.882379) (end 55.04 30.2) (width 1) (layer "F.Cu") (net 2))
@@
   (segment (start 35.8 44.9) (end 35.654649 45.045351) (width 1) (layer "B.Cu") (net 19))
   (segment (start 41.065 35.435) (end 38.1 38.4) (width 1) (layer "F.Cu") (net 25))
-  (segment (start 63.085 23.815) (end 51.685 23.815) (width 1) (layer "F.Cu") (net 25))
   (segment (start 21.7 38.4) (end 21.71 38.41) (width 1) (layer "F.Cu") (net 25))
-  (segment (start 75.04 21.9) (end 75.04 26.16) (width 1) (layer "F.Cu") (net 25))
   (segment (start 49.81 25.09) (end 42.41 25.09) (width 1) (layer "F.Cu") (net 25))
+  (segment (start 70.817621 30.382379) (end 67.6 30.382379) (width 1) (layer "F.Cu") (net 25))
   (segment (start 51.685 23.815) (end 50.785 23.815) (width 1) (layer "F.Cu") (net 25))
   (segment (start 52.56 22.94) (end 51.685 23.815) (width 1) (layer "F.Cu") (net 25))
   (segment (start 42.41 25.09) (end 41.065 26.435) (width 1) (layer "F.Cu") (net 25))
+  (segment (start 75.8 25.4) (end 70.817621 30.382379) (width 1) (layer "F.Cu") (net 25))
   (segment (start 49.81 25.09) (end 49.81 40.88) (width 1) (layer "F.Cu") (net 25))
-  (segment (start 65 21.9) (end 63.085 23.815) (width 1) (layer "F.Cu") (net 25))
+  (segment (start 75.8 21.8) (end 75.8 25.4) (width 1) (layer "F.Cu") (net 25))
+  (segment (start 51.685 23.815) (end 63.085 23.815) (width 1) (layer "F.Cu") (net 25))
   (segment (start 21.71 38.41) (end 21.71 41.365) (width 1) (layer "F.Cu") (net 25))
+  (segment (start 65.1 21.8) (end 75.8 21.8) (width 1) (layer "F.Cu") (net 25))
+  (segment (start 63.085 23.815) (end 65.1 21.8) (width 1) (layer "F.Cu") (net 25))
   (segment (start 41.065 26.435) (end 37.017024 26.435) (width 1) (layer "F.Cu") (net 25))
   (segment (start 38.1 38.4) (end 21.7 38.4) (width 1) (layer "F.Cu") (net 25))
-  (segment (start 75.04 26.16) (end 70.817621 30.382379) (width 1) (layer "F.Cu") (net 25))
   (segment (start 52.56 20.5) (end 52.56 22.94) (width 1) (layer "F.Cu") (net 25))
-  (segment (start 70.817621 30.382379) (end 67.6 30.382379) (width 1) (layer "F.Cu") (net 25))
-  (segment (start 75.04 21.9) (end 65 21.9) (width 1) (layer "F.Cu") (net 25))
   (segment (start 50.785 23.815) (end 49.6 25) (width 1) (layer "F.Cu") (net 25))
   (segment (start 67.6 30.382379) (end 67.6 30.8) (width 1) (layer "F.Cu") (net 25))
@@
   (segment (start 34.477024 26.899999) (end 34.477024 25.677024) (width 1) (layer "B.Cu") (net 31))
   (segment (start 26.9 18.47) (end 25.28 20.09) (width 1) (layer "F.Cu") (net 32))
-  (segment (start 63.6 20.5) (end 55.1 20.5) (width 1) (layer "F.Cu") (net 32))
   (segment (start 25.28 22.71) (end 24.46 23.53) (width 1) (layer "F.Cu") (net 32))
+  (segment (start 64.6 19.5) (end 63.6 20.5) (width 1) (layer "F.Cu") (net 32))
   (segment (start 26.9 18.4) (end 26.9 18.47) (width 1) (layer "F.Cu") (net 32))
-  (segment (start 77 19.5) (end 64.6 19.5) (width 1) (layer "F.Cu") (net 32))
-  (segment (start 74.995 34.63) (end 74.995 34.105) (width 1) (layer "F.Cu") (net 32))
   (segment (start 21.49 22.4) (end 18.6 25.29) (width 1) (layer "F.Cu") (net 32))
   (segment (start 44.117621 29.9) (end 44.117621 41.582379) (width 1) (layer "F.Cu") (net 32))
-  (segment (start 79.1 21.6) (end 77 19.5) (width 1) (layer "F.Cu") (net 32))
+  (segment (start 79.1 30) (end 79.1 21.6) (width 1) (layer "F.Cu") (net 32))
   (segment (start 25.59 22.4) (end 21.49 22.4) (width 1) (layer "F.Cu") (net 32))
   (segment (start 24.46 23.53) (end 24.46 29.835) (width 1) (layer "F.Cu") (net 32))
   (segment (start 27.914649 16.653002) (end 27.914649 17.385351) (width 1) (layer "F.Cu") (net 32))
   (segment (start 27.914649 17.385351) (end 26.9 18.4) (width 1) (layer "F.Cu") (net 32))
-  (segment (start 64.6 19.5) (end 63.6 20.5) (width 1) (layer "F.Cu") (net 32))
+  (segment (start 77 19.5) (end 64.6 19.5) (width 1) (layer "F.Cu") (net 32))
+  (segment (start 75.785 34.58) (end 75.785 33.315) (width 1) (layer "F.Cu") (net 32))
+  (segment (start 75.785 33.315) (end 79.1 30) (width 1) (layer "F.Cu") (net 32))
   (segment (start 22.894649 46.705351) (end 22.894649 47.263002) (width 1) (layer "F.Cu") (net 32))
   (segment (start 25.28 20.09) (end 25.28 22.71) (width 1) (layer "F.Cu") (net 32))
   (segment (start 27 43.6) (end 25.3 45.3) (width 1) (layer "F.Cu") (net 32))
-  (segment (start 74.995 34.105) (end 79.1 30) (width 1) (layer "F.Cu") (net 32))
   (segment (start 42.1 43.6) (end 27 43.6) (width 1) (layer "F.Cu") (net 32))
+  (segment (start 63.6 20.5) (end 55.1 20.5) (width 1) (layer "F.Cu") (net 32))
   (segment (start 24.46 29.835) (end 27.49 32.865) (width 1) (layer "F.Cu") (net 32))
-  (segment (start 79.1 30) (end 79.1 21.6) (width 1) (layer "F.Cu") (net 32))
   (segment (start 25.3 45.3) (end 24.3 45.3) (width 1) (layer "F.Cu") (net 32))
   (segment (start 44.117621 41.582379) (end 42.1 43.6) (width 1) (layer "F.Cu") (net 32))
+  (segment (start 79.1 21.6) (end 77 19.5) (width 1) (layer "F.Cu") (net 32))
   (segment (start 24.3 45.3) (end 22.894649 46.705351) (width 1) (layer "F.Cu") (net 32))
   (segment (start 55.1 21.8) (end 52 24.9) (width 1) (layer "B.Cu") (net 32))
